File: MUNIN 100.kicad_sch (KiCad schematic)
At the start: 78 parts, among them IC1 ACHS-7123, J1 TX_IN, J2 Conn_Coaxial, J3 Molex kk 2.54-3, J4 Conn_01x01_Pin, J5 Conn_01x01_Pin, Q1 ISS55EP06LMXTSA1, Q2 MRF101AN, Q3 MRF101BN, U2 LM358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

Commit message: kicad10 update, minor schematic changes
Other:
- note added: "Bias 100 mA per transistor ?"
- note added: "Q1 is soldered upside down"
- moved on the sheet: C2, C8, R1, R4, RV1, RV2
